File: pcbs/right_thumb.kicad_pcb (KiCad board)
At the start: 2 copper layers, 43.7 x 43.7 mm, 9 parts

Commit message: Update right_thumb.kicad_pcb
rotated stabilizer footprint on left thumb to avoid stablilizer wire interfering with mounting hole
Routing:
- net T_COL: track 45.2 -> 46.7 mm
